Commit message: refactor(kinematics): enforce single-source robot contract

File: ros2_ws/src/robot_description/urdf/jackal.urdf.xacro (robot description, xacro)
@@ -2,7 +2,28 @@
 <robot xmlns:xacro="http://www.ros.org/wiki/xacro" name="jackal">
   <xacro:arg name="prefix" default=""/>
+  <xacro:arg name="wheel_radius" default=""/>
+  <xacro:arg name="wheel_width" default=""/>
+  <xacro:arg name="geometric_track_width" default=""/>
+  <xacro:arg name="wheelbase" default=""/>
+  <xacro:arg name="base_mass" default=""/>
+  <xacro:arg name="wheel_mass" default=""/>
+  <xacro:arg name="front_left_joint_name" default=""/>
+  <xacro:arg name="front_right_joint_name" default=""/>
+  <xacro:arg name="rear_left_joint_name" default=""/>
+  <xacro:arg name="rear_right_joint_name" default=""/>
   <xacro:include filename="jackal_base.xacro"/>
   <xacro:include filename="jackal_sensors.xacro"/>
-  <xacro:jackal_base prefix="$(arg prefix)"/>
+  <xacro:jackal_base
+      prefix="$(arg prefix)"
+      wheel_radius="$(arg wheel_radius)"
+      wheel_width="$(arg wheel_width)"
+      geometric_track_width="$(arg geometric_track_width)"
+      wheelbase="$(arg wheelbase)"
+      base_mass="$(arg base_mass)"
+      wheel_mass="$(arg wheel_mass)"
+      front_left_joint_name="$(arg front_left_joint_name)"
+      front_right_joint_name="$(arg front_right_joint_name)"
+      rear_left_joint_name="$(arg rear_left_joint_name)"
+      rear_right_joint_name="$(arg rear_right_joint_name)"/>
   <xacro:jackal_sensors prefix="$(arg prefix)"/>
 </robot>

File: ros2_ws/src/robot_description/urdf/jackal_base.xacro (robot description, xacro)
@@ -1,9 +1,10 @@
 <?xml version="1.0"?>
 <robot xmlns:xacro="http://www.ros.org/wiki/xacro">
-  <xacro:macro name="jackal_wheel" params="prefix name x y">
-    <link name="${prefix}${name}_wheel_link">
+  <xacro:macro name="jackal_wheel"
+               params="prefix position_name joint_name x y wheel_radius wheel_width wheel_mass">
+    <link name="${prefix}${position_name}_wheel_link">
       <inertial>
         <origin xyz="0 0 0" rpy="0 0 0"/>
-        <mass value="0.477"/>
+        <mass value="${wheel_mass}"/>
         <inertia ixx="0.000286" ixy="0" ixz="0"
                  iyy="0.002290" iyz="0" izz="0.002290"/>
@@ -12,5 +13,5 @@
         <origin xyz="0 0 0" rpy="1.57079632679 0 0"/>
         <geometry>
-          <cylinder radius="0.098" length="0.040"/>
+          <cylinder radius="${wheel_radius}" length="${wheel_width}"/>
         </geometry>
         <material name="jackal_tire">
@@ -21,21 +22,24 @@
         <origin xyz="0 0 0" rpy="1.57079632679 0 0"/>
         <geometry>
-          <cylinder radius="0.098" length="0.040"/>
+          <cylinder radius="${wheel_radius}" length="${wheel_width}"/>
         </geometry>
       </collision>
     </link>
-    <joint name="${prefix}${name}_wheel_joint" type="continuous">
+    <!-- JointState names are the exact robot-YAML contract.  A visual-link
+         prefix must never silently rename the controller/odometry joints. -->
+    <joint name="${joint_name}" type="continuous">
       <origin xyz="${x} ${y} 0.0345" rpy="0 0 0"/>
       <parent link="${prefix}base_link"/>
-      <child link="${prefix}${name}_wheel_link"/>
+      <child link="${prefix}${position_name}_wheel_link"/>
       <axis xyz="0 1 0"/>
       <dynamics damping="0.05" friction="0.0"/>
     </joint>
   </xacro:macro>
-  <xacro:macro name="jackal_base" params="prefix:=''">
+  <xacro:macro name="jackal_base"
+               params="prefix wheel_radius wheel_width geometric_track_width wheelbase base_mass wheel_mass front_left_joint_name front_right_joint_name rear_left_joint_name rear_right_joint_name">
     <link name="${prefix}base_link">
       <inertial>
         <origin xyz="0 0 0.10" rpy="0 0 0"/>
-        <mass value="17.0"/>
+        <mass value="${base_mass}"/>
         <inertia ixx="0.25" ixy="0" ixz="0"
                  iyy="0.35" iyz="0" izz="0.45"/>
@@ -57,8 +61,32 @@
       </collision>
     </link>
-    <xacro:jackal_wheel prefix="${prefix}" name="front_left" x="0.131" y="0.187795"/>
-    <xacro:jackal_wheel prefix="${prefix}" name="front_right" x="0.131" y="-0.187795"/>
-    <xacro:jackal_wheel prefix="${prefix}" name="rear_left" x="-0.131" y="0.187795"/>
-    <xacro:jackal_wheel prefix="${prefix}" name="rear_right" x="-0.131" y="-0.187795"/>
+    <xacro:jackal_wheel
+        prefix="${prefix}" position_name="front_left"
+        joint_name="${front_left_joint_name}"
+        x="${float(wheelbase) / 2.0}"
+        y="${float(geometric_track_width) / 2.0}"
+        wheel_radius="${wheel_radius}" wheel_width="${wheel_width}"
+        wheel_mass="${wheel_mass}"/>
+    <xacro:jackal_wheel
+        prefix="${prefix}" position_name="front_right"
+        joint_name="${front_right_joint_name}"
+        x="${float(wheelbase) / 2.0}"
+        y="${-float(geometric_track_width) / 2.0}"
+        wheel_radius="${wheel_radius}" wheel_width="${wheel_width}"
+        wheel_mass="${wheel_mass}"/>
+    <xacro:jackal_wheel
+        prefix="${prefix}" position_name="rear_left"
+        joint_name="${rear_left_joint_name}"
+        x="${-float(wheelbase) / 2.0}"
+        y="${float(geometric_track_width) / 2.0}"
+        wheel_radius="${wheel_radius}" wheel_width="${wheel_width}"
+        wheel_mass="${wheel_mass}"/>
+    <xacro:jackal_wheel
+        prefix="${prefix}" position_name="rear_right"
+        joint_name="${rear_right_joint_name}"
+        x="${-float(wheelbase) / 2.0}"
+        y="${-float(geometric_track_width) / 2.0}"
+        wheel_radius="${wheel_radius}" wheel_width="${wheel_width}"
+        wheel_mass="${wheel_mass}"/>
   </xacro:macro>
 </robot>
